Commit message: fix: requested changes

File: my_robot/urdf/my_robot.xacro (robot description, xacro)
@@ -21,5 +21,5 @@
       <origin xyz="0 0 0" rpy=" 0 0 0"/>
       <geometry>
-        <box size=".4 .2 .1"/>
+        <box size=".5 .2 .1"/>
       </geometry>
     </collision>
@@ -27,5 +27,5 @@
       <origin xyz="0 0 0" rpy=" 0 0 0"/>
       <geometry>
-        <box size=".4 .2 .1"/>
+        <box size=".5 .2 .1"/>
       </geometry>
     </visual>
@@ -33,5 +33,5 @@
       <origin xyz="-0.15 0 -0.05" rpy=" 0 0 0"/>
       <geometry>
-        <sphere radius="0.0499"/>
+        <sphere radius="0.0999"/>
       </geometry>
     </collision>
@@ -39,5 +39,5 @@
       <origin xyz="-0.15 0 -0.05" rpy=" 0 0 0"/>
       <geometry>
-        <sphere radius="0.05"/>
+        <sphere radius="0.1"/>
       </geometry>
     </visual>
@@ -45,5 +45,5 @@
       <origin xyz="0.15 0 -0.05" rpy=" 0 0 0"/>
       <geometry>
-        <sphere radius="0.0499"/>
+        <sphere radius="0.0999"/>
       </geometry>
     </collision>
@@ -51,5 +51,5 @@
       <origin xyz="0.15 0 -0.05" rpy=" 0 0 0"/>
       <geometry>
-        <sphere radius="0.05"/>
+        <sphere radius="0.1"/>
       </geometry>
     </visual>
@@ -69,5 +69,5 @@
       <origin xyz="0 0 0" rpy="0 1.5707 1.5707" />
       <geometry>
-        <cylinder radius="0.1" length="0.05" />
+        <cylinder radius="0.15" length="0.07" />
       </geometry>
     </collision>
@@ -75,5 +75,5 @@
       <origin xyz="0 0 0" rpy="0 1.5707 1.5707" />
       <geometry>
-        <cylinder radius="0.1" length="0.05" />
+        <cylinder radius="0.15" length="0.07" />
       </geometry>
     </visual>
@@ -92,5 +92,5 @@
       <origin xyz="0 0 0" rpy="0 1.5707 1.5707" />
       <geometry>
-        <cylinder radius="0.1" length="0.05" />
+        <cylinder radius="0.15" length="0.07" />
       </geometry>
     </collision>
@@ -98,5 +98,5 @@
       <origin xyz="0 0 0" rpy="0 1.5707 1.5707" />
       <geometry>
-        <cylinder radius="0.1" length="0.05" />
+        <cylinder radius="0.15" length="0.07" />
       </geometry>
     </visual>
@@ -142,5 +142,5 @@
   <joint type="fixed" name="camera_joint">
     <axis xyz="0 1 0" rpy="0 0 0" />
-    <origin xyz="0.2 0 0" rpy="0 0 0" />
+    <origin xyz="0.25 0 0" rpy="0 0 0" />
     <parent link="chassis" />
     <child link="camera" />
@@ -169,5 +169,5 @@
   <joint type="fixed" name="hokuyo_joint">
     <axis xyz="0 1 0" />
-    <origin  xyz="0.15 0 0.1" rpy="0 0 0" />
+    <origin  xyz="0.2 0 0.07" rpy="0 0 0" />
     <parent link="chassis" />
     <child  link="hokuyo" />
@@ -175,17 +175,17 @@
   <!-- COLORS -->
   <gazebo reference="chassis">
-    <material>Gazebo/Blue</material>
+    <material>Gazebo/Brown</material>
   </gazebo>
   <gazebo reference="left_wheel">
-    <material>Gazebo/Green</material>
+    <material>Gazebo/Black</material>
   </gazebo>
   <gazebo reference="right_wheel">
-    <material>Gazebo/Green</material>
+    <material>Gazebo/Black</material>
   </gazebo>
   <gazebo reference="camera">
-    <material>Gazebo/Red</material>
+    <material>Gazebo/White</material>
   </gazebo>
   <gazebo reference="hokuyo">
-    <material>Gazebo/Grey</material>
+    <material>Gazebo/Yellow</material>
   </gazebo>
 </robot>
